Commit message: 로봇이 충돌로 넘어져 뒹굴던 문제 수정 — 충돌체 제거(기구학 구동에 맞춤)
앞서 세 링크 모두 중력을 꺼서 '가라앉다 튕겨 날아가는' 경로는 막았지만,
이번엔 사람·장애물과 접촉하는 순간 뒤집혀 공중에서 뒹구는 일이 생겼다.
(실측: 접촉 후 z=3.37m, roll 98°, pitch 83°)

원인: URDF 의 <kinematic>true</kinematic> 가 **아무 효과가 없다.**
gz-sim8 라이브러리에 'kinematic' 문자열 자체가 없어 태그가 조용히 무시되고,
링크는 완전한 동역학 강체로 취급된다. 중력까지 꺼둔 상태라 충돌 충격이
감쇠 없이 그대로 남아 한 번 부딪히면 영구히 회전·상승한다.

이 로봇은 VelocityControl 로 속도를 직접 지정해 움직인다(바퀴도 시각 전용).
즉 충돌체를 둬도 로봇을 막아주지 못하고 충격만 받는다. 얻는 것 없이
넘어짐만 유발하므로 base_link/turret_link/gun_link 의 collision 을 제거했다.

- 장애물 회피는 LiDAR + Nav2 코스트맵이 전담한다(원래도 그랬다).
- GpuLidar 는 렌더링 기반이라 visual 을 보므로 감지에 영향 없다.
- 트레이드오프: Nav2 가 잘못 계획하면 로봇이 벽을 물리적으로 통과한다.
  대신 넘어지거나 날아가서 임무가 통째로 망가지는 일은 없어진다.

검증: 주행 중 z=0.150000 고정, roll/pitch=0 유지.
조난자 등록 (5.9,0.9) GT(6,1) 오차 0.14m / (8.8,-7.6) 은 누운 자세(L1)라
모델 원점 기준 1.3m — 몸통 길이(1.7m)를 감안하면 정상 범위.

File: src/ugv_description/urdf/ugv.urdf.xacro (robot description, xacro)
@@ -18,7 +18,14 @@
       <material name="silver"/>
     </visual>
-    <collision name="base_collision">
-      <geometry><box size="0.50 0.34 0.14"/></geometry>
-    </collision>
+    <!-- collision 없음 — 의도적.
+         이 로봇은 VelocityControl 로 속도를 직접 지정해 움직인다(기구학 구동,
+         바퀴도 시각 전용). 그런데 gz-sim8 은 <kinematic> 태그를 읽지 않아서
+         (libgz-sim8 에 해당 문자열 자체가 없음) 링크가 완전한 동역학 강체로
+         취급된다. 중력까지 꺼둔 상태라 충돌 충격이 감쇠 없이 그대로 남아,
+         한 번 부딪히면 영구히 회전·상승해 로봇이 공중에서 뒹군다.
+         (실측: 벽/장애물 접촉 후 z=3.4m, roll 98°, pitch 83°)
+         충돌체를 두어도 기구학 구동이라 어차피 로봇을 막아주지 못하고
+         충격만 받는다. 장애물 회피는 전적으로 LiDAR + Nav2 코스트맵이 담당한다.
+         GpuLidar 는 렌더링 기반이라 visual 을 보므로 감지에도 영향이 없다. -->
     <inertial>
       <mass value="5.0"/>
@@ -79,7 +86,5 @@
       <material name="silver"/>
     </visual>
-    <collision>
-      <geometry><box size="0.06 0.12 0.30"/></geometry>
-    </collision>
+    <!-- collision 없음 — base_link 주석 참조 (기구학 구동이라 충격만 받음) -->
     <inertial>
       <mass value="1.0"/>
@@ -101,8 +106,5 @@
       <material name="gray"/>
     </visual>
-    <collision>
-      <origin xyz="0.03 0 -0.02" rpy="0 0 0"/>
-      <geometry><box size="0.08 0.08 0.06"/></geometry>
-    </collision>
+    <!-- collision 없음 — base_link 주석 참조 -->
     <inertial>
       <mass value="0.2"/>

Commit message: feat(모델): URDF 에 로봇 접두사 인자 추가 — 2대 동시 스폰 준비
한 월드에 로봇을 둘 띄우려면 TF 프레임과 gz 센서 토픽이 로봇마다 달라야
한다. xacro 인자 prefix 를 넣어 이름을 갈래로 만든다.

  prefix=""       기존과 완전히 동일 (1대 구성 그대로)
  prefix="ugv1/"  ugv1/base_footprint, /ugv1/scan, /ugv1/cmd_vel ...

★ cmd_vel 과 odom 은 반드시 절대경로로 명시해야 한다.
상대 토픽으로 두면 모델 스코프가 아니라 루트로 해석된다(실측: gz topic -l
에서 /cmd_vel, /odom 으로 나옴). 접두사가 없으면 두 로봇이 같은 /cmd_vel 을
받아 나란히 똑같이 움직인다.

바퀴 매크로의 매개변수 prefix 는 side 로 바꿨다. 좌우 구분과 로봇 구분이
같은 이름이라 헷갈렸다.

회귀 검증(prefix 비운 상태로 큰 월드 실행):
  gz 토픽 이름 기존과 동일 (/cmd_vel /odom /scan /joint_states /turret_*)
  /scan 9.65Hz, /odom 49.1Hz — 기존 9.8Hz/50Hz 와 같은 수준
  TF 는 map → odom 으로 접두사 없음
  로봇 주행 정상 (6초에 (-1.5,-1.8) → (-0.3,-4.9))

xacro 출력 비교에서 예전과 다른 줄은 위 절대경로 두 곳뿐이다.

File: src/ugv_description/urdf/ugv.urdf.xacro (robot description, xacro)
@@ -1,4 +1,13 @@
 <?xml version="1.0"?>
 <robot name="ugv" xmlns:xacro="http://www.ros.org/wiki/xacro">
+  <!-- 로봇 2대를 한 월드에 띄우기 위한 접두사.
+       비워 두면 지금까지와 완전히 같은 이름이 나온다(1대 구성 그대로).
+       'ugv1/' 처럼 주면 TF 프레임은 ugv1/base_footprint, gz 센서 토픽은
+       /ugv1/scan 이 된다.
+       gz 토픽을 반드시 명시해야 하는 이유: 상대 토픽(cmd_vel, odom)이
+       모델 스코프가 아니라 루트로 해석된다(실측 gz topic -l 에서 /cmd_vel).
+       접두사를 안 붙이면 두 로봇이 같은 /cmd_vel 을 받아 함께 움직인다. -->
+  <xacro:arg name="prefix" default=""/>
+  <xacro:property name="P" value="$(arg prefix)"/>
   <material name="black"><color rgba="0.1 0.1 0.1 1"/></material>
   <material name="dark_gray"><color rgba="0.3 0.3 0.3 1"/></material>
@@ -7,11 +16,11 @@
   <material name="blue"><color rgba="0.0 0.0 0.8 1"/></material>
   <material name="red"><color rgba="0.8 0.0 0.0 1"/></material>
-  <link name="base_footprint"/>
+  <link name="${P}base_footprint"/>
   <joint name="base_joint" type="fixed">
-    <parent link="base_footprint"/>
-    <child link="base_link"/>
+    <parent link="${P}base_footprint"/>
+    <child link="${P}base_link"/>
     <origin xyz="0 0 0.15" rpy="0 0 0"/>
   </joint>
-  <link name="base_link">
+  <link name="${P}base_link">
     <visual>
       <geometry><box size="0.50 0.34 0.14"/></geometry>
@@ -40,16 +49,18 @@
        바닥에 닿는 순간 튕기는데 base 에는 중력이 없어 되돌아오지 못한다.
        → 로봇이 공중으로 날아가 뒤집힌다. 반드시 세 링크 모두 꺼야 한다. -->
-  <gazebo reference="base_link">
+  <gazebo reference="${P}base_link">
     <kinematic>true</kinematic>
     <gravity>false</gravity>
   </gazebo>
-  <gazebo reference="turret_link">
+  <gazebo reference="${P}turret_link">
     <gravity>false</gravity>
   </gazebo>
-  <gazebo reference="gun_link">
+  <gazebo reference="${P}gun_link">
     <gravity>false</gravity>
   </gazebo>
-  <xacro:macro name="wheel" params="prefix x_reflect y_reflect">
-    <link name="${prefix}_wheel_link">
+  <!-- 매개변수 이름이 'side' 인 이유: 로봇 구분 접두사 P 와 헷갈리지 않게.
+       예전엔 이 자리도 prefix 였다. -->
+  <xacro:macro name="wheel" params="side x_reflect y_reflect">
+    <link name="${P}${side}_wheel_link">
       <visual>
         <origin xyz="0 0 0" rpy="1.570796 0 0"/>
@@ -58,17 +69,17 @@
       </visual>
     </link>
-    <joint name="${prefix}_wheel_joint" type="fixed">
-      <parent link="base_link"/>
-      <child link="${prefix}_wheel_link"/>
+    <joint name="${P}${side}_wheel_joint" type="fixed">
+      <parent link="${P}base_link"/>
+      <child link="${P}${side}_wheel_link"/>
       <origin xyz="${0.20 * x_reflect} ${0.19 * y_reflect} -0.10" rpy="0 0 0"/>
     </joint>
   </xacro:macro>
-  <xacro:wheel prefix="front_left" x_reflect="1" y_reflect="1" />
-  <xacro:wheel prefix="front_right" x_reflect="1" y_reflect="-1" />
-  <xacro:wheel prefix="mid_left" x_reflect="0" y_reflect="1" />
-  <xacro:wheel prefix="mid_right" x_reflect="0" y_reflect="-1" />
-  <xacro:wheel prefix="rear_left" x_reflect="-1" y_reflect="1" />
-  <xacro:wheel prefix="rear_right" x_reflect="-1" y_reflect="-1" />
-  <link name="laser_frame">
+  <xacro:wheel side="front_left" x_reflect="1" y_reflect="1" />
+  <xacro:wheel side="front_right" x_reflect="1" y_reflect="-1" />
+  <xacro:wheel side="mid_left" x_reflect="0" y_reflect="1" />
+  <xacro:wheel side="mid_right" x_reflect="0" y_reflect="-1" />
+  <xacro:wheel side="rear_left" x_reflect="-1" y_reflect="1" />
+  <xacro:wheel side="rear_right" x_reflect="-1" y_reflect="-1" />
+  <link name="${P}laser_frame">
     <visual>
       <geometry><cylinder radius="0.035" length="0.04"/></geometry>
@@ -77,9 +88,9 @@
   </link>
   <joint name="laser_joint" type="fixed">
-    <parent link="base_link"/>
-    <child link="laser_frame"/>
+    <parent link="${P}base_link"/>
+    <child link="${P}laser_frame"/>
     <origin xyz="0.245 0.0 0.08" rpy="0 0 3.14159265"/>
   </joint>
-  <link name="turret_link">
+  <link name="${P}turret_link">
     <visual>
       <geometry><box size="0.06 0.12 0.30"/></geometry>
@@ -94,11 +105,11 @@
   </link>
   <joint name="turret_yaw_joint" type="revolute">
-    <parent link="base_link"/>
-    <child link="turret_link"/>
+    <parent link="${P}base_link"/>
+    <child link="${P}turret_link"/>
     <origin xyz="0 0 0.245" rpy="0 0 0"/>
     <axis xyz="0 0 1"/>
     <limit lower="-6.2832" upper="6.2832" effort="100" velocity="1.0"/>
   </joint>
-  <link name="gun_link">
+  <link name="${P}gun_link">
     <visual>
       <origin xyz="0.03 0 -0.02" rpy="0 0 0"/>
@@ -114,11 +125,11 @@
   </link>
   <joint name="turret_pitch_joint" type="revolute">
-    <parent link="turret_link"/>
-    <child link="gun_link"/>
+    <parent link="${P}turret_link"/>
+    <child link="${P}gun_link"/>
     <origin xyz="0 0 0.15" rpy="0 0 0"/>
     <axis xyz="0 1 0"/>
     <limit lower="-0.52" upper="0.52" effort="100" velocity="1.0"/>
   </joint>
-  <link name="camera_link">
+  <link name="${P}camera_link">
     <visual>
       <geometry><box size="0.025 0.09 0.025"/></geometry>
@@ -127,21 +138,24 @@
   </link>
   <joint name="camera_joint" type="fixed">
-    <parent link="gun_link"/>
-    <child link="camera_link"/>
+    <parent link="${P}gun_link"/>
+    <child link="${P}camera_link"/>
     <origin xyz="0.06 0.0 0.01" rpy="0 0 0"/>
   </joint>
   <gazebo>
     <plugin filename="gz-sim-joint-state-publisher-system" name="gz::sim::systems::JointStatePublisher">
-      <topic>/joint_states</topic>
-    </plugin>
+      <topic>/${P}joint_states</topic>
+    </plugin>
+    <!-- cmd_vel 과 odom 은 상대 토픽으로 두면 모델 스코프가 아니라 루트로
+         해석된다(실측). 접두사를 안 붙이면 두 로봇이 같은 /cmd_vel 을 받아
+         나란히 움직인다. 반드시 명시한다. -->
     <plugin filename="gz-sim-velocity-control-system" name="gz::sim::systems::VelocityControl">
-      <topic>cmd_vel</topic>
+      <topic>/${P}cmd_vel</topic>
     </plugin>
     <plugin filename="gz-sim-odometry-publisher-system" name="gz::sim::systems::OdometryPublisher">
-      <odom_frame>odom</odom_frame>
-      <robot_base_frame>base_footprint</robot_base_frame>
+      <odom_frame>${P}odom</odom_frame>
+      <robot_base_frame>${P}base_footprint</robot_base_frame>
       <odom_publish_frequency>50</odom_publish_frequency>
-      <odom_topic>odom</odom_topic>
-      <tf_topic>/model/ugv/tf</tf_topic>
+      <odom_topic>/${P}odom</odom_topic>
+      <tf_topic>/model/${P}ugv/tf</tf_topic>
       <publish_tf>false</publish_tf>
     </plugin>
@@ -149,18 +163,18 @@
       <joint_name>turret_yaw_joint</joint_name>
       <use_velocity_commands>true</use_velocity_commands>
-      <topic>/turret_yaw_cmd</topic>
+      <topic>/${P}turret_yaw_cmd</topic>
     </plugin>
     <plugin filename="gz-sim-joint-controller-system" name="gz::sim::systems::JointController">
       <joint_name>turret_pitch_joint</joint_name>
       <use_velocity_commands>true</use_velocity_commands>
-      <topic>/turret_pitch_cmd</topic>
-    </plugin>
-  </gazebo>
-  <gazebo reference="laser_frame">
+      <topic>/${P}turret_pitch_cmd</topic>
+    </plugin>
+  </gazebo>
+  <gazebo reference="${P}laser_frame">
     <sensor name="lidar" type="gpu_lidar">
       <pose>0 0 0 0 0 0</pose>
-      <topic>/scan</topic>
+      <topic>/${P}scan</topic>
       <update_rate>10</update_rate>
-      <gz_frame_id>laser_frame</gz_frame_id>
+      <gz_frame_id>${P}laser_frame</gz_frame_id>
       <ray>
         <scan>
@@ -182,13 +196,13 @@
     </sensor>
   </gazebo>
-  <gazebo reference="camera_link">
+  <gazebo reference="${P}camera_link">
     <sensor name="rgbd_camera" type="rgbd_camera">
       <pose>0 0 0 0 0 0</pose>
-      <topic>/camera</topic>
+      <topic>/${P}camera</topic>
       <!-- 포인트클라우드를 Nav2 장애물 입력으로 쓰려면 frame_id 가 TF 에
            있는 이름이어야 한다. 없으면 스코프명(ugv/base_footprint/...)이
            나가고 코스트맵이 변환을 못 해 통째로 버린다.
            (열화상도 같은 이유로 이미 지정돼 있다) -->
-      <gz_frame_id>camera_link</gz_frame_id>
+      <gz_frame_id>${P}camera_link</gz_frame_id>
       <update_rate>15</update_rate>
       <camera>
@@ -214,10 +228,10 @@
        주의: thermal 센서는 ogre2 렌더 엔진에서만 동작 (월드 sensors 플러그인 render_engine=ogre2 필요).
        출력: /thermal/image_raw (16bit mono, 픽셀값 = 온도[K] / linear_resolution). -->
-  <gazebo reference="camera_link">
+  <gazebo reference="${P}camera_link">
     <sensor name="thermal_camera" type="thermal">
       <pose>0 0 0 0 0 0</pose>
-      <topic>/thermal/image_raw</topic>
+      <topic>/${P}thermal/image_raw</topic>
       <update_rate>10</update_rate>
-      <gz_frame_id>camera_link</gz_frame_id>
+      <gz_frame_id>${P}camera_link</gz_frame_id>
       <camera>
         <horizontal_fov>1.089</horizontal_fov>
